Commit message: 修复roslaunch报错找不到STL文件的错误

File: inspire_hand_description/robots/inspire_hand_left.urdf (robot description, URDF)
Before this commit: robot inspire_hand_left, 22 links, 21 joints
Links:
- link Link1: geometry collision mesh filename=package://inspire_hand_description/meshes/left/arm_Link1.STL; visual mesh filename=package://inspire_hand_description/meshes/left/arm_Link1.STL
- link Link2: geometry collision mesh filename=package://inspire_hand_description/meshes/left/arm_Link2.STL; visual mesh filename=package://inspire_hand_description/meshes/left/arm_Link2.STL
- link Link3: geometry collision mesh filename=package://inspire_hand_description/meshes/left/arm_Link3.STL; visual mesh filename=package://inspire_hand_description/meshes/left/arm_Link3.STL
- link Link4: geometry collision mesh filename=package://inspire_hand_description/meshes/left/arm_Link4.STL; visual mesh filename=package://inspire_hand_description/meshes/left/arm_Link4.STL
- link Link5: geometry collision mesh filename=package://inspire_hand_description/meshes/left/arm_Link5.STL; visual mesh filename=package://inspire_hand_description/meshes/left/arm_Link5.STL
- link Link6: geometry collision mesh filename=package://inspire_hand_description/meshes/left/arm_Link6.STL; visual mesh filename=package://inspire_hand_description/meshes/left/arm_Link6.STL
